Commit message: upgrade urdf model

File: gyrosse_description/urdf/gazebo.xacro (robot description, xacro)
@@ -1,4 +1,4 @@
 <?xml version="1.0" ?>
-<robot name="URDF_Gyrosse" xmlns:xacro="http://www.ros.org/wiki/xacro" >
+<robot name="gyrosse" xmlns:xacro="http://www.ros.org/wiki/xacro" >
 <xacro:property name="body_color" value="Gazebo/Silver" />
 <gazebo reference="base_link">
@@ -9,5 +9,12 @@
   <gravity>true</gravity>
 </gazebo>
-<gazebo reference="wheel_right_1">
+<gazebo reference="chassis">
+  <material>${body_color}</material>
+  <mu1>0.2</mu1>
+  <mu2>0.2</mu2>
+  <self_collide>true</self_collide>
+  <gravity>true</gravity>
+</gazebo>
+<gazebo reference="right_wheel">
   <material>${body_color}</material>
   <mu1>0.2</mu1>
@@ -15,5 +22,5 @@
   <self_collide>true</self_collide>
 </gazebo>
-<gazebo reference="flywheel_right_1">
+<gazebo reference="right_flywheel">
   <material>${body_color}</material>
   <mu1>0.2</mu1>
@@ -21,5 +28,5 @@
   <self_collide>true</self_collide>
 </gazebo>
-<gazebo reference="wheel_left_1">
+<gazebo reference="left_wheel">
   <material>${body_color}</material>
   <mu1>0.2</mu1>
@@ -27,5 +34,5 @@
   <self_collide>true</self_collide>
 </gazebo>
-<gazebo reference="flywheel_left_1">
+<gazebo reference="left_flywheel">
   <material>${body_color}</material>
   <mu1>0.2</mu1>

File: gyrosse_description/urdf/gyrosse_description.xacro (robot description, xacro)
@@ -15,5 +15,5 @@
     <origin xyz="0 0 0" rpy="0 0 0"/>
     <geometry>
-      <mesh filename="file://$(find URDF_Gyrosse_description)/meshes/base_link.stl" scale="0.001 0.001 0.001"/>
+      <mesh filename="file://$(find gyrosse_description)/meshes/chassis.stl" scale="0.001 0.001 0.001"/>
     </geometry>
     <material name="silver"/>
@@ -22,5 +22,5 @@
     <origin xyz="0 0 0" rpy="0 0 0"/>
     <geometry>
-      <mesh filename="file://$(find URDF_Gyrosse_description)/meshes/base_link.stl" scale="0.001 0.001 0.001"/>
+      <mesh filename="file://$(find gyrosse_description)/meshes/chassis.stl" scale="0.001 0.001 0.001"/>
     </geometry>
   </collision>
@@ -41,5 +41,5 @@
     <origin xyz="0 0 0" rpy="0 0 0"/>
     <geometry>
-      <mesh filename="file://$(find URDF_Gyrosse_description)/meshes/right_wheel.stl" scale="0.001 0.001 0.001"/>
+      <mesh filename="file://$(find gyrosse_description)/meshes/right_wheel.stl" scale="0.001 0.001 0.001"/>
     </geometry>
     <material name="Black"/>
@@ -48,5 +48,5 @@
     <origin xyz="0 0 0" rpy="0 0 0"/>
     <geometry>
-      <mesh filename="file://$(find URDF_Gyrosse_description)/meshes/right_wheel.stl" scale="0.001 0.001 0.001"/>
+      <mesh filename="file://$(find gyrosse_description)/meshes/right_wheel.stl" scale="0.001 0.001 0.001"/>
     </geometry>
   </collision>
@@ -68,5 +68,5 @@
     <origin xyz="-0.108 0 0" rpy="0 0 0"/>
     <geometry>
-      <mesh filename="file://$(find URDF_Gyrosse_description)/meshes/right_flywheel.stl" scale="0.001 0.001 0.001"/>
+      <mesh filename="file://$(find gyrosse_description)/meshes/right_flywheel.stl" scale="0.001 0.001 0.001"/>
     </geometry>
     <material name="Grey"/>
@@ -75,5 +75,5 @@
     <origin xyz="-0.108 0 0" rpy="0 0 0"/>
     <geometry>
-      <mesh filename="file://$(find URDF_Gyrosse_description)/meshes/right_flywheel.stl" scale="0.001 0.001 0.001"/>
+      <mesh filename="file://$(find gyrosse_description)/meshes/right_flywheel.stl" scale="0.001 0.001 0.001"/>
     </geometry>
   </collision>
@@ -95,5 +95,5 @@
     <origin xyz="-0.381 0 0" rpy="0 0 0"/>
     <geometry>
-      <mesh filename="file://$(find URDF_Gyrosse_description)/meshes/left_wheel.stl" scale="0.001 0.001 0.001"/>
+      <mesh filename="file://$(find gyrosse_description)/meshes/left_wheel.stl" scale="0.001 0.001 0.001"/>
     </geometry>
     <material name="Black"/>
@@ -102,5 +102,5 @@
     <origin xyz="-0.381 0 0" rpy="0 0 0"/>
     <geometry>
-      <mesh filename="file://$(find URDF_Gyrosse_description)/meshes/left_wheel.stl" scale="0.001 0.001 0.001"/>
+      <mesh filename="file://$(find gyrosse_description)/meshes/left_wheel.stl" scale="0.001 0.001 0.001"/>
     </geometry>
   </collision>
@@ -122,5 +122,5 @@
     <origin xyz="-0.273 0 0" rpy="0 0 0"/>
     <geometry>
-      <mesh filename="file://$(find URDF_Gyrosse_description)/meshes/left_flywheel.stl" scale="0.001 0.001 0.001"/>
+      <mesh filename="file://$(find gyrosse_description)/meshes/left_flywheel.stl" scale="0.001 0.001 0.001"/>
     </geometry>
     <material name="Grey"/>
@@ -129,5 +129,5 @@
     <origin xyz="-0.273 0 0" rpy="0 0 0"/>
     <geometry>
-      <mesh filename="file://$(find URDF_Gyrosse_description)/meshes/left_flywheel.stl" scale="0.001 0.001 0.001"/>
+      <mesh filename="file://$(find gyrosse_description)/meshes/left_flywheel.stl" scale="0.001 0.001 0.001"/>
     </geometry>
   </collision>

File: gyrosse_description/urdf/materials.xacro (robot description, xacro)
@@ -1,4 +1,4 @@
 <?xml version="1.0" ?>
-<robot name="URDF_Gyrosse" xmlns:xacro="http://www.ros.org/wiki/xacro" >
+<robot name="gyrosse" xmlns:xacro="http://www.ros.org/wiki/xacro" >
 <material name="silver">
   <color rgba="0.700 0.700 0.700 1.000"/>

File: gyrosse_description/urdf/ros2_control.xacro (robot description, xacro)
@@ -1,24 +1,23 @@
 <?xml version="1.0" ?>
-<robot name="URDF_Gyrosse" xmlns:xacro="http://www.ros.org/wiki/xacro" >
+<robot name="gyrosse" xmlns:xacro="http://www.ros.org/wiki/xacro" >
 <ros2_control name="GazeboSystem" type="system">
     <hardware>
       <plugin>gazebo_ros2_control/GazeboSystem</plugin>
     </hardware>
-    <joint name="right_wheel">
+    <joint name="right_wheel_joint">
       <command_interface name="velocity"/>
       <state_interface name="position"/>
       <state_interface name="velocity"/>
     </joint>
-    <joint name="left_wheel">
+    <joint name="left_wheel_joint">
       <command_interface name="velocity"/>
       <state_interface name="position"/>
       <state_interface name="velocity"/>
     </joint>
-    <joint name="right_flywheel">
+    <joint name="right_flywheel_joint">
       <command_interface name="velocity"/>
-      </command_interface>
       <state_interface name="velocity"/>
     </joint>
-    <joint name="left_flywheel">
+    <joint name="left_flywheel_joint">
       <command_interface name="velocity"/>
       <state_interface name="velocity"/>
@@ -27,5 +26,5 @@
   <gazebo>
     <plugin filename="libgazebo_ros2_control.so" name="gazebo_ros2_control">
-      <parameters>$(find URDF_Gyrosse_description)/config/gyrosse_drive_controller.yaml</parameters>
+      <parameters>$(find gyrosse_bringup)/config/gyrosse_controller.yaml</parameters>
     </plugin>
   </gazebo>

Commit message: interne

File: gyrosse_description/urdf/gazebo.xacro (robot description, xacro)
@@ -3,11 +3,4 @@
 <xacro:property name="body_color" value="Gazebo/Silver" />
 <gazebo reference="base_link">
-  <material>${body_color}</material>
-  <mu1>0.2</mu1>
-  <mu2>0.2</mu2>
-  <self_collide>true</self_collide>
-  <gravity>true</gravity>
-</gazebo>
-<gazebo reference="chassis">
   <material>${body_color}</material>
   <mu1>0.2</mu1>

File: gyrosse_description/urdf/gyrosse_description.xacro (robot description, xacro)
@@ -4,7 +4,6 @@
 <xacro:include filename="$(find gyrosse_description)/urdf/gazebo.xacro" />
 <xacro:include filename="$(find gyrosse_description)/urdf/ros2_control.xacro" />
- <link name="base_link" />
 <!-- Chassis -->
-<link name="chassis">
+<link name="base_link">
   <inertial>
     <origin xyz="0.19050000000000009 -0.007676917492127958 -0.0014829191458506099" rpy="0 0 0"/>
@@ -26,9 +25,4 @@
   </collision>
 </link>
-<joint name="chassis_joint" type="fixed">
-  <origin xyz="0 0 0" rpy="0 0 0" />
-  <parent link="base_link" />
-  <child link="chassis" />
-</joint>
 <!-- right wheel Link -->
 <link name="right_wheel">
@@ -54,5 +48,5 @@
 <joint name="right_wheel_joint" type="continuous">
   <origin xyz="0 0 0" rpy="0 0 0"/>
-  <parent link="chassis"/>
+  <parent link="base_link"/>
   <child link="right_wheel"/>
   <axis xyz="0 0 0"/>
@@ -81,5 +75,5 @@
 <joint name="right_flywheel_joint" type="continuous">
   <origin xyz="0.108 0 0" rpy="0 0 0"/>
-  <parent link="chassis"/>
+  <parent link="base_link"/>
   <child link="right_flywheel"/>
   <axis xyz="1 0 0"/>
@@ -135,5 +129,5 @@
 <joint name="left_flywheel_joint" type="continuous">
   <origin xyz="0.273 0 0" rpy="0 0 0"/>
-  <parent link="chassis"/>
+  <parent link="base_link"/>
   <child link="left_flywheel"/>
   <axis xyz="-1 0 0"/>

Commit message: ros2_control parameter

File: gyrosse_description/urdf/gazebo.xacro (robot description, xacro)
@@ -1,35 +1,23 @@
 <?xml version="1.0" ?>
-<robot name="gyrosse" xmlns:xacro="http://www.ros.org/wiki/xacro" >
-<xacro:property name="body_color" value="Gazebo/Silver" />
-<gazebo reference="base_link">
-  <material>${body_color}</material>
-  <mu1>0.2</mu1>
-  <mu2>0.2</mu2>
-  <self_collide>true</self_collide>
-  <gravity>true</gravity>
-</gazebo>
-<gazebo reference="right_wheel">
-  <material>${body_color}</material>
-  <mu1>0.2</mu1>
-  <mu2>0.2</mu2>
-  <self_collide>true</self_collide>
-</gazebo>
-<gazebo reference="right_flywheel">
-  <material>${body_color}</material>
-  <mu1>0.2</mu1>
-  <mu2>0.2</mu2>
-  <self_collide>true</self_collide>
-</gazebo>
-<gazebo reference="left_wheel">
-  <material>${body_color}</material>
-  <mu1>0.2</mu1>
-  <mu2>0.2</mu2>
-  <self_collide>true</self_collide>
-</gazebo>
-<gazebo reference="left_flywheel">
-  <material>${body_color}</material>
-  <mu1>0.2</mu1>
-  <mu2>0.2</mu2>
-  <self_collide>true</self_collide>
-</gazebo>
+<robot name="gyrosse" xmlns:xacro="http://www.ros.org/wiki/xacro">
+<xacro:property name="package_name" value="gyrosse_description"/>
+<xacro:include filename="$(find ${package_name})/urdf/include/gazebo_macros.xacro" />
+<xacro:gazebo_default name="base_link"
+            color="Gazebo/Silver"/>
+<xacro:gazebo_default name="motor_wheel_right"
+            color="Gazebo/Black"/>
+<xacro:gazebo_default name="motor_wheel_left"
+            color="Gazebo/Black"/>
+<xacro:gazebo_default name="motor_flywheel_right"
+            color="Gazebo/Black"/>
+<xacro:gazebo_default name="motor_flywheel_left"
+            color="Gazebo/Black"/>
+<xacro:gazebo_default name="flywheel_right"
+            color="Gazebo/Orange"/>
+<xacro:gazebo_default name="flywheel_left"
+            color="Gazebo/Orange"/>
+<xacro:gazebo_default name="wheel_right"
+            color="Gazebo/Grey"/>
+<xacro:gazebo_default name="wheel_left"
+            color="Gazebo/Grey"/>
 </robot>

File: gyrosse_description/urdf/gyrosse_description.xacro (robot description, xacro)
@@ -1,135 +1,21 @@
 <?xml version="1.0" ?>
 <robot name="gyrosse" xmlns:xacro="http://www.ros.org/wiki/xacro">
-<xacro:include filename="$(find gyrosse_description)/urdf/materials.xacro" />
-<xacro:include filename="$(find gyrosse_description)/urdf/gazebo.xacro" />
-<xacro:include filename="$(find gyrosse_description)/urdf/ros2_control.xacro" />
-<!-- Chassis -->
-<link name="base_link">
-  <inertial>
-    <origin xyz="0.19050000000000009 -0.007676917492127958 -0.0014829191458506099" rpy="0 0 0"/>
-    <mass value="13.254937098226266"/>
-    <inertia ixx="0.132414" iyy="0.271154" izz="0.221585" ixy="0" iyz="0.000151" ixz="0"/>
-  </inertial>
-  <visual>
-    <origin xyz="0 0 0" rpy="0 0 0"/>
-    <geometry>
-      <mesh filename="file://$(find gyrosse_description)/meshes/chassis.stl" scale="0.001 0.001 0.001"/>
-    </geometry>
-    <material name="silver"/>
-  </visual>
-  <collision>
-    <origin xyz="0 0 0" rpy="0 0 0"/>
-    <geometry>
-      <mesh filename="file://$(find gyrosse_description)/meshes/chassis.stl" scale="0.001 0.001 0.001"/>
-    </geometry>
-  </collision>
-</link>
-<!-- right wheel Link -->
-<link name="right_wheel">
-  <inertial>
-    <origin xyz="-0.049489111284257994 -1.3199520432358287e-15 2.061614684425312e-16" rpy="0 0 0"/>
-    <mass value="1.2625898797377435"/>
-    <inertia ixx="0.041938" iyy="0.021235" izz="0.021235" ixy="0" iyz="0" ixz="0"/>
-  </inertial>
-  <visual>
-    <origin xyz="0 0 0" rpy="0 0 0"/>
-    <geometry>
-      <mesh filename="file://$(find gyrosse_description)/meshes/right_wheel.stl" scale="0.001 0.001 0.001"/>
-    </geometry>
-    <material name="Black"/>
-  </visual>
-  <collision>
-    <origin xyz="0 0 0" rpy="0 0 0"/>
-    <geometry>
-      <mesh filename="file://$(find gyrosse_description)/meshes/right_wheel.stl" scale="0.001 0.001 0.001"/>
-    </geometry>
-  </collision>
-</link>
-<joint name="right_wheel_joint" type="continuous">
-  <origin xyz="0 0 0" rpy="0 0 0"/>
-  <parent link="base_link"/>
-  <child link="right_wheel"/>
-  <axis xyz="0 0 0"/>
-</joint>
-<!-- right flywheel Link -->
-<link name="right_flywheel">
-  <inertial>
-    <origin xyz="-0.008066340570656319 1.271316816228521e-16 1.7394980092897013e-16" rpy="0 0 0"/>
-    <mass value="1.7384117767470415"/>
-    <inertia ixx="0.018431" iyy="0.009354" izz="0.009354" ixy="0" iyz="0" ixz="0"/>
-  </inertial>
-  <visual>
-    <origin xyz="-0.108 0 0" rpy="0 0 0"/>
-    <geometry>
-      <mesh filename="file://$(find gyrosse_description)/meshes/right_flywheel.stl" scale="0.001 0.001 0.001"/>
-    </geometry>
-    <material name="Grey"/>
-  </visual>
-  <collision>
-    <origin xyz="-0.108 0 0" rpy="0 0 0"/>
-    <geometry>
-      <mesh filename="file://$(find gyrosse_description)/meshes/right_flywheel.stl" scale="0.001 0.001 0.001"/>
-    </geometry>
-  </collision>
-</link>
-<joint name="right_flywheel_joint" type="continuous">
-  <origin xyz="0.108 0 0" rpy="0 0 0"/>
-  <parent link="base_link"/>
-  <child link="right_flywheel"/>
-  <axis xyz="1 0 0"/>
-</joint>
-  <!-- left wheel Link -->
-<link name="left_wheel">
-  <inertial>
-    <origin xyz="0.04948911128425798 -8.531713599697203e-16 -2.7715603505479613e-16" rpy="0 0 0"/>
-    <mass value="1.2625898797377435"/>
-    <inertia ixx="0.041938" iyy="0.021235" izz="0.021235" ixy="0" iyz="0" ixz="0"/>
-  </inertial>
-  <visual>
-    <origin xyz="-0.381 0 0" rpy="0 0 0"/>
-    <geometry>
-      <mesh filename="file://$(find gyrosse_description)/meshes/left_wheel.stl" scale="0.001 0.001 0.001"/>
-    </geometry>
-    <material name="Black"/>
-  </visual>
-  <collision>
-    <origin xyz="-0.381 0 0" rpy="0 0 0"/>
-    <geometry>
-      <mesh filename="file://$(find gyrosse_description)/meshes/left_wheel.stl" scale="0.001 0.001 0.001"/>
-    </geometry>
-  </collision>
-</link>
-<joint name="left_wheel_joint" type="continuous">
-  <origin xyz="0.381 0 0" rpy="0 0 0"/>
-  <parent link="base_link"/>
-  <child link="left_wheel"/>
-  <axis xyz="1 0 0"/>
-</joint>
-<!-- left flywheel Link -->
-<link name="left_flywheel">
-  <inertial>
-    <origin xyz="0.008066340570656305 1.553831664279304e-16 -1.0733641945145496e-16" rpy="0 0 0"/>
-    <mass value="1.7384117767470415"/>
-    <inertia ixx="0.018431" iyy="0.009354" izz="0.009354" ixy="0" iyz="0" ixz="0"/>
-  </inertial>
-  <visual>
-    <origin xyz="-0.273 0 0" rpy="0 0 0"/>
-    <geometry>
-      <mesh filename="file://$(find gyrosse_description)/meshes/left_flywheel.stl" scale="0.001 0.001 0.001"/>
-    </geometry>
-    <material name="Grey"/>
-  </visual>
-  <collision>
-    <origin xyz="-0.273 0 0" rpy="0 0 0"/>
-    <geometry>
-      <mesh filename="file://$(find gyrosse_description)/meshes/left_flywheel.stl" scale="0.001 0.001 0.001"/>
-    </geometry>
-  </collision>
-</link>
-<joint name="left_flywheel_joint" type="continuous">
-  <origin xyz="0.273 0 0" rpy="0 0 0"/>
-  <parent link="base_link"/>
-  <child link="left_flywheel"/>
-  <axis xyz="-1 0 0"/>
-</joint>
+<xacro:property name="package_name" value="gyrosse_description"/>
+<xacro:include filename="$(find ${package_name})/urdf/include/common_macros.xacro" />
+<xacro:include filename="$(find ${package_name})/urdf/include/materials.xacro" />
+<xacro:include filename="$(find ${package_name})/urdf/gazebo.xacro" />
+<xacro:include filename="$(find ${package_name})/urdf/ros2_control.xacro" />
+<xacro:chassis name="base_link"/>
+<xacro:motor_wheel name="motor_wheel_right"
+                   joint_origin_xyz="-0.145 0.06 0.04" joint_rpy="0 0 0"/>
+<xacro:motor_wheel name="motor_wheel_left"
+                   joint_origin_xyz="0.145 0.06 -0.04" joint_rpy="0 ${pi} 0"/>
+<xacro:motor_flywheel name="motor_flywheel_right"
+                      joint_origin_xyz="-0.125 0.06 0.04" joint_rpy="0 0 0"/>
+<xacro:motor_flywheel name="motor_flywheel_left"
+                      joint_origin_xyz="0.125 0.06 -0.04" joint_rpy="0 ${pi} 0"/>
+<xacro:flywheel name="flywheel_right"/>
+<xacro:flywheel name="flywheel_left"/>
+<xacro:wheel name="wheel_right"/>
+<xacro:wheel name="wheel_left"/>
 </robot>

File: gyrosse_description/urdf/include/materials.xacro (robot description, xacro)
@@ -1,17 +1,17 @@
 <?xml version="1.0" ?>
-<robot name="gyrosse" xmlns:xacro="http://www.ros.org/wiki/xacro" >
+<robot xmlns:xacro="http://www.ros.org/wiki/xacro" >
 <material name="silver">
   <color rgba="0.700 0.700 0.700 1.000"/>
 </material>
- <material name="Black">
+ <material name="black">
     <color rgba="0 0 0 1" />
   </material>
-  <material name="Grey">
+  <material name="grey">
     <color rgba="0.8 0.8 0.8 1" />
   </material>
-  <material name="Orange">
+  <material name="orange">
     <color rgba="1 0.6 0 1" />
   </material>
-  <material name="White">
+  <material name="white">
     <color rgba="1 1 1 1" />
   </material>

File: gyrosse_description/urdf/ros2_control.xacro (robot description, xacro)
@@ -1,25 +1,67 @@
 <?xml version="1.0" ?>
 <robot name="gyrosse" xmlns:xacro="http://www.ros.org/wiki/xacro" >
-<ros2_control name="GazeboSystem" type="system">
+<ros2_control name="gyrosse_ros2_control" type="system">
     <hardware>
-      <plugin>gazebo_ros2_control/GazeboSystem</plugin>
+      <plugin>myactuator_hardware_interface/MyActuatorHardwareInterface</plugin>
     </hardware>
-    <joint name="right_wheel_joint">
-      <command_interface name="velocity"/>
-      <state_interface name="position"/>
-      <state_interface name="velocity"/>
+    <joint name="joint_flywheel_right">
+          <param name="ifname">"can0"</param>
+          <param name="can_id">1</param>
+          <param name="timeout">0.1</param>
+          <param name="position_acceleration">200000</param>
+          <param name="position_deceleration">200000</param>
+          <param name="velocity_acceleration">200000</param>
+          <param name="velocity_deceleration">200000</param>
+          <param name="kp_current">50</param>
+          <param name="ki_current">50</param>
+          <param name="kp_speed">100</param>
+          <param name="ki_speed">5</param>
+          <param name="kp_position">100</param>
+          <param name="ki_position">0</param>
     </joint>
-    <joint name="left_wheel_joint">
-      <command_interface name="velocity"/>
-      <state_interface name="position"/>
-      <state_interface name="velocity"/>
+    <joint name="joint_flywheel_left">
+          <param name="ifname">"can0"</param>
+          <param name="can_id">2</param>
+          <param name="timeout">0.1</param>
+          <param name="position_acceleration">200000</param>
+          <param name="position_deceleration">200000</param>
+          <param name="velocity_acceleration">200000</param>
+          <param name="velocity_deceleration">200000</param>
+          <param name="kp_current">50</param>
+          <param name="ki_current">50</param>
+          <param name="kp_speed">100</param>
+          <param name="ki_speed">5</param>
+          <param name="kp_position">100</param>
+          <param name="ki_position">0</param>
     </joint>
-    <joint name="right_flywheel_joint">
-      <command_interface name="velocity"/>
-      <state_interface name="velocity"/>
+    <joint name="joint_wheel_right">
+          <param name="ifname">"can0"</param>
+          <param name="can_id">3</param>
+          <param name="timeout">0.1</param>
+          <param name="position_acceleration">200000</param>
+          <param name="position_deceleration">200000</param>
+          <param name="velocity_acceleration">200000</param>
+          <param name="velocity_deceleration">200000</param>
+          <param name="kp_current">50</param>
+          <param name="ki_current">50</param>
+          <param name="kp_speed">100</param>
+          <param name="ki_speed">5</param>
+          <param name="kp_position">100</param>
+          <param name="ki_position">0</param>
     </joint>
-    <joint name="left_flywheel_joint">
-      <command_interface name="velocity"/>
-      <state_interface name="velocity"/>
+    <joint name="joint_wheel_left">
+          <param name="ifname">"can0"</param>
+          <param name="can_id">4</param>
+          <param name="timeout">0.1</param>
+          <param name="position_acceleration">200000</param>
+          <param name="position_deceleration">200000</param>
+          <param name="velocity_acceleration">200000</param>
+          <param name="velocity_deceleration">200000</param>
+          <param name="kp_current">50</param>
+          <param name="ki_current">50</param>
+          <param name="kp_speed">100</param>
+          <param name="ki_speed">5</param>
+          <param name="kp_position">100</param>
+          <param name="ki_position">0</param>
     </joint>
   </ros2_control>
