Commit message: change syntax can0

File: gyrosse_description/urdf/ros2_control.xacro (robot description, xacro)
@@ -6,5 +6,5 @@
     </hardware>
     <joint name="joint_flywheel_right">
-          <param name="ifname">"can0"</param>
+          <param name="ifname">can0</param>
           <param name="can_id">1</param>
           <param name="timeout">0.1</param>
@@ -21,5 +21,5 @@
     </joint>
     <joint name="joint_flywheel_left">
-          <param name="ifname">"can0"</param>
+          <param name="ifname">can0</param>
           <param name="can_id">2</param>
           <param name="timeout">0.1</param>
@@ -35,6 +35,6 @@
           <param name="ki_position">0</param>
     </joint>
-    <joint name="joint_wheel_right">
-          <param name="ifname">"can0"</param>
+<joint name="joint_wheel_right">
+          <param name="ifname">can0</param>
           <param name="can_id">3</param>
           <param name="timeout">0.1</param>
@@ -51,5 +51,5 @@
     </joint>
     <joint name="joint_wheel_left">
-          <param name="ifname">"can0"</param>
+          <param name="ifname">can0</param>
           <param name="can_id">4</param>
           <param name="timeout">0.1</param>
