Commit message: gyrosse model upgrade

File: gyrosse_description/urdf/gyrosse.ros2_control.xacro (robot description, xacro)
@@ -1,25 +1,15 @@
 <?xml version="1.0" ?>
 <robot xmlns:xacro="http://www.ros.org/wiki/xacro" >
-  <xacro:macro name="ros2_control" params="
-    ifname_can
-    use_fake_hardware:=false
-    fake_sensor_commands:=false
-    ">
-      <ros2_control name="gyrosse_ros2_control" type="system">
+  <xacro:macro name="ros2_control" params="name prefix ifname">
+      <ros2_control name="${name}_wheel_ros2_control" type="system">
         <hardware>
-          <xacro:if value="${use_fake_hardware}">
-            <plugin>mock_components/GenericSystem</plugin>
-            <param name="mock_sensor_commands">${fake_sensor_commands}</param>
-            <param name="state_following_offset">0.0</param>
-          </xacro:if>
-          <xacro:unless value="${use_fake_hardware}">
             <plugin>myactuator_hardware_interface/MyActuatorHardwareInterface</plugin>
-            <param name="ifname">${ifname_can}</param>
-          </xacro:unless>
+            <param name="ifname">${ifname}</param>
+            <param name="timeout">1000</param>
+            <param name="max_speed">2000</param>
         </hardware>
-<joint name="joint_wheel_right">
+        <joint name="${prefix}left_wheel_joint">
               <param name="can_id">1</param>
-              <param name="timeout">1000</param>
-              <param name="reducer_ratio">6.2/1</param>
+              <param name="reducer_ratio">6.2</param>
               <param name="speed_constant">30</param>
               <param name="torque_constant">0.29</param>
@@ -29,15 +19,14 @@
               <param name="velocity_acceleration">20000</param>
               <param name="velocity_deceleration">20000</param>
-              <param name="kp_current">50</param>
-              <param name="ki_current">50</param>
+              <param name="kp_current">100</param>
+              <param name="ki_current">100</param>
               <param name="kp_speed">100</param>
-              <param name="ki_speed">5</param>
+              <param name="ki_speed">50</param>
               <param name="kp_position">100</param>
               <param name="ki_position">0</param>
         </joint>
-        <joint name="joint_wheel_left">
+        <joint name="${prefix}right_wheel_joint">
               <param name="can_id">2</param>
-              <param name="timeout">1000</param>
-              <param name="reducer_ratio">6.2/1</param>
+              <param name="reducer_ratio">6.2</param>
               <param name="speed_constant">30</param>
               <param name="torque_constant">0.29</param>
@@ -47,10 +36,10 @@
               <param name="velocity_acceleration">20000</param>
               <param name="velocity_deceleration">20000</param>
-              <param name="kp_current">50</param>
-              <param name="ki_current">50</param>
+              <param name="kp_current">100</param>
+              <param name="ki_current">100</param>
               <param name="kp_speed">100</param>
-              <param name="ki_speed">5</param>
+              <param name="ki_speed">50</param>
               <param name="kp_position">100</param>
-              <param name="ki_position">0</param>
+              <param name="ki_position">0.0</param>
         </joint>
 <!--

Commit message: add flywheel cmd

File: gyrosse_description/urdf/gyrosse.ros2_control.xacro (robot description, xacro)
@@ -7,5 +7,5 @@
             <param name="ifname">${ifname}</param>
             <param name="timeout">1000</param>
-            <param name="max_speed">2000</param>
+            <param name="max_speed">5000</param>
         </hardware>
         <joint name="${prefix}left_wheel_joint">
@@ -43,9 +43,8 @@
               <param name="ki_position">0.0</param>
         </joint>
-<!--
-        <joint name="joint_flywheel_right">
-              <param name="can_id">1</param>
+        <joint name="${prefix}left_flywheel_joint">
+              <param name="can_id">3</param>
               <param name="timeout">1000</param>
-              <param name="reducer_ratio">9/1</param>
+              <param name="reducer_ratio">9</param>
               <param name="speed_constant">30</param>
               <param name="torque_constant">0.29</param>
@@ -62,8 +61,8 @@
               <param name="ki_position">0</param>
         </joint>
-        <joint name="joint_flywheel_left">
-              <param name="can_id">2</param>
+        <joint name="${prefix}right_flywheel_joint">
+              <param name="can_id">4</param>
               <param name="timeout">1000</param>
-              <param name="reducer_ratio">9/1</param>
+              <param name="reducer_ratio">9</param>
               <param name="speed_constant">30</param>
               <param name="torque_constant">0.29</param>
@@ -80,5 +79,4 @@
               <param name="ki_position">0</param>
         </joint>
--->
       </ros2_control>
       <gazebo>
